File: 3V3-Supply.kicad_sch (KiCad schematic)
At the start: 8 parts, among them IC1 ADP2301AUJZ-R7

Commit message: some placement and IMPORTANT schematic mistake fix from heirarchichal label importing
Parts:
- C6: footprint robot-cortex:C_0402_1005Metric -> esp32-socket-switcher:C_0402_1005Metric; symbol robot-cortex:Capacitor -> esp32-socket-switcher:Capacitor
- C7, C8: footprint robot-cortex:C_0603_1608Metric -> esp32-socket-switcher:C_0603_1608Metric; symbol robot-cortex:Capacitor -> esp32-socket-switcher:Capacitor
- D1: footprint robot-cortex:SOD2512X110N -> esp32-socket-switcher:SOD2512X110N
- IC1: footprint robot-cortex:SOT95P280X100-6N -> esp32-socket-switcher:SOT95P280X100-6N; symbol robot-cortex:ADP2301AUJZ-R7 -> esp32-socket-switcher:ADP2301AUJZ-R7
- L1: symbol robot-cortex:L -> esp32-socket-switcher:L
- R4: footprint robot-cortex:R_0402_1005Metric -> esp32-socket-switcher:R_0402_1005Metric; symbol robot-cortex:Resistor -> esp32-socket-switcher:Resistor
Changed lines of the file:
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@@
     (effects (font (size 1.27 1.27)) (justify left))
   )
-  (symbol (lib_id "robot-cortex:Resistor") (at 160.02 100.33 0) (mirror x) (unit 1)
+  (symbol (lib_id "esp32-socket-switcher:Resistor") (at 160.02 100.33 0) (mirror x) (unit 1)
     (in_bom yes) (on_board yes) (dnp no)
     (property "Reference" "R4" (at 157.1316 99.695 0)
@@
       (effects (font (size 1.27 1.27)) (justify right))
     )
-    (property "Footprint" "robot-cortex:R_0402_1005Metric" (at 154.94 113.03 0)
+    (property "Footprint" "esp32-socket-switcher:R_0402_1005Metric" (at 154.94 113.03 0)
       (effects (font (size 1.27 1.27)) hide)
     )
@@
     (pin "2")
     (instances
-      (project "robot-cortex"
+      (project "esp32-socket-switcher"
         (path "/19e4cb9f-d0a4-4ce0-8aa4-5fe95563dc37"
           (reference "R4") (unit 1)
@@
     )
   )
-  (symbol (lib_id "robot-cortex:Resistor") (at 160.02 90.17 0) (mirror x) (unit 1)
+  (symbol (lib_id "esp32-socket-switcher:Resistor") (at 160.02 90.17 0) (mirror x) (unit 1)
     (in_bom yes) (on_board yes) (dnp no)
     (property "Reference" "R4" (at 157.1316 89.535 0)
@@
       (effects (font (size 1.27 1.27)) (justify right))
     )
-    (property "Footprint" "robot-cortex:R_0402_1005Metric" (at 154.94 102.87 0)
+    (property "Footprint" "esp32-socket-switcher:R_0402_1005Metric" (at 154.94 102.87 0)
       (effects (font (size 1.27 1.27)) hide)
     )
@@
     (pin "2")
     (instances
-      (project "robot-cortex"
+      (project "esp32-socket-switcher"
         (path "/19e4cb9f-d0a4-4ce0-8aa4-5fe95563dc37"
           (reference "R4") (unit 1)
@@
     (pin "")
     (instances
-      (project "robot-cortex"
+      (project "esp32-socket-switcher"
         (path "/19e4cb9f-d0a4-4ce0-8aa4-5fe95563dc37/2757805a-b362-411e-a4a6-92c934b4db34"
           (reference "#PWR015") (unit 1)
@@
       (effects (font (size 1.27 1.27)) (justify left))
     )
-    (property "Footprint" "robot-cortex:SOD2512X110N" (at 47.32 96.52 0)
+    (property "Footprint" "esp32-socket-switcher:SOD2512X110N" (at 47.32 96.52 0)
       (effects (font (size 1.27 1.27)) (justify left top) hide)
     )
@@
     (pin "2")
     (instances
-      (project "robot-cortex"
+      (project "esp32-socket-switcher"
         (path "/19e4cb9f-d0a4-4ce0-8aa4-5fe95563dc37/2757805a-b362-411e-a4a6-92c934b4db34"
           (reference "D1") (unit 1)
@@
     (pin "")
     (instances
-      (project "robot-cortex"
+      (project "esp32-socket-switcher"
         (path "/19e4cb9f-d0a4-4ce0-8aa4-5fe95563dc37/2757805a-b362-411e-a4a6-92c934b4db34"
           (reference "#PWR019") (unit 1)
@@
     (pin "")
     (instances
-      (project "robot-cortex"
+      (project "esp32-socket-switcher"
         (path "/19e4cb9f-d0a4-4ce0-8aa4-5fe95563dc37/2757805a-b362-411e-a4a6-92c934b4db34"
           (reference "#PWR016") (unit 1)
@@
     )
   )
-  (symbol (lib_id "robot-cortex:Capacitor") (at 113.03 73.66 90) (unit 1)
+  (symbol (lib_id "esp32-socket-switcher:Capacitor") (at 113.03 73.66 90) (unit 1)
     (in_bom yes) (on_board yes) (dnp no)
     (property "Reference" "C6" (at 112.776 71.501 0)
@@
       (effects (font (size 1.27 1.27)) (justify left bottom))
     )
-    (property "Footprint" "robot-cortex:C_0402_1005Metric" (at 116.84 72.6948 0)
+    (property "Footprint" "esp32-socket-switcher:C_0402_1005Metric" (at 116.84 72.6948 0)
       (effects (font (size 1.27 1.27)) hide)
     )
@@
     (pin "2")
     (instances
-      (project "robot-cortex"
+      (project "esp32-socket-switcher"
         (path "/19e4cb9f-d0a4-4ce0-8aa4-5fe95563dc37/2757805a-b362-411e-a4a6-92c934b4db34"
           (reference "C6") (unit 1)
@@
     )
   )
-  (symbol (lib_id "robot-cortex:Capacitor") (at 168.91 87.63 0) (unit 1)
+  (symbol (lib_id "esp32-socket-switcher:Capacitor") (at 168.91 87.63 0) (unit 1)
     (in_bom yes) (on_board yes) (dnp no)
     (property "Reference" "C7" (at 170.815 88.519 0)
@@
       (effects (font (size 1.27 1.27)) (justify left bottom) hide)
     )
-    (property "Footprint" "robot-cortex:C_0603_1608Metric" (at 169.8752 91.44 0)
+    (property "Footprint" "esp32-socket-switcher:C_0603_1608Metric" (at 169.8752 91.44 0)
       (effects (font (size 1.27 1.27)) hide)
     )
@@
     (pin "2")
     (instances
-      (project "robot-cortex"
+      (project "esp32-socket-switcher"
         (path "/19e4cb9f-d0a4-4ce0-8aa4-5fe95563dc37/2757805a-b362-411e-a4a6-92c934b4db34"
           (reference "C7") (unit 1)
@@
     (pin "")
     (instances
-      (project "robot-cortex"
+      (project "esp32-socket-switcher"
         (path "/19e4cb9f-d0a4-4ce0-8aa4-5fe95563dc37/2757805a-b362-411e-a4a6-92c934b4db34"
           (reference "#PWR018") (unit 1)
@@
     (pin "")
     (instances
-      (project "robot-cortex"
+      (project "esp32-socket-switcher"
         (path "/19e4cb9f-d0a4-4ce0-8aa4-5fe95563dc37/2757805a-b362-411e-a4a6-92c934b4db34"
           (reference "#PWR03") (unit 1)
@@
     (pin "")
     (instances
-      (project "robot-cortex"
+      (project "esp32-socket-switcher"
         (path "/19e4cb9f-d0a4-4ce0-8aa4-5fe95563dc37/2757805a-b362-411e-a4a6-92c934b4db34"
           (reference "#PWR017") (unit 1)
@@
     )
   )
-  (symbol (lib_id "robot-cortex:ADP2301AUJZ-R7") (at 101.6 85.09 0) (unit 1)
+  (symbol (lib_id "esp32-socket-switcher:ADP2301AUJZ-R7") (at 101.6 85.09 0) (unit 1)
     (in_bom yes) (on_board yes) (dnp no) (fields_autoplaced)
     (property "Reference" "IC1" (at 114.3 77.343 0)
@@
       (effects (font (size 1.27 1.27)))
     )
-    (property "Footprint" "robot-cortex:SOT95P280X100-6N" (at 123.19 180.01 0)
+    (property "Footprint" "esp32-socket-switcher:SOT95P280X100-6N" (at 123.19 180.01 0)
       (effects (font (size 1.27 1.27)) (justify left top) hide)
     )
@@
     (pin "6")
     (instances
-      (project "robot-cortex"
+      (project "esp32-socket-switcher"
         (path "/19e4cb9f-d0a4-4ce0-8aa4-5fe95563dc37/2757805a-b362-411e-a4a6-92c934b4db34"
           (reference "IC1") (unit 1)
@@
     )
   )
-  (symbol (lib_id "robot-cortex:Capacitor") (at 176.53 87.63 0) (unit 1)
+  (symbol (lib_id "esp32-socket-switcher:Capacitor") (at 176.53 87.63 0) (unit 1)
     (in_bom yes) (on_board yes) (dnp no)
     (property "Reference" "C8" (at 178.435 88.519 0)
@@
       (effects (font (size 1.27 1.27)) (justify left bottom) hide)
     )
-    (property "Footprint" "robot-cortex:C_0603_1608Metric" (at 177.4952 91.44 0)
+    (property "Footprint" "esp32-socket-switcher:C_0603_1608Metric" (at 177.4952 91.44 0)
       (effects (font (size 1.27 1.27)) hide)
     )
@@
     (pin "2")
     (instances
-      (project "robot-cortex"
+      (project "esp32-socket-switcher"
         (path "/19e4cb9f-d0a4-4ce0-8aa4-5fe95563dc37/2757805a-b362-411e-a4a6-92c934b4db34"
           (reference "C8") (unit 1)
@@
     )
   )
-  (symbol (lib_id "robot-cortex:L") (at 152.4 83.82 90) (unit 1)
+  (symbol (lib_id "esp32-socket-switcher:L") (at 152.4 83.82 90) (unit 1)
     (in_bom yes) (on_board yes) (dnp no) (fields_autoplaced)
     (property "Reference" "L1" (at 152.4 78.74 90)
@@
     (pin "2")
     (instances
-      (project "robot-cortex"
+      (project "esp32-socket-switcher"
         (path "/19e4cb9f-d0a4-4ce0-8aa4-5fe95563dc37/2757805a-b362-411e-a4a6-92c934b4db34"
           (reference "L1") (unit 1)
