File: esp32-socket-switcher.kicad_pcb (KiCad board)
At the start: 4 copper layers, 49.8 x 34.5 mm, 45 parts, among them IC1 ADP2301AUJZ-R7, J1 USB4110GFA, J2 4DB-P108-06, K1 G5CA-1A DC5, Q1 SS8050-G, Q2 SS8050-G, Q3 CSD17575Q3T, U2 ESP32-WROOM-32E-H4, U5 CP2102N-A02-GQFN24R

Commit message: routed
Parts:
- moved J2 2.41 mm to (78.8, 65.7)
Routing:
- net /AC_LIVE: track 16.1 -> 20.0 mm
- net /SWITCH_IN: track 32.6 -> 35.1 mm
- net /AC_LIVE_SWITCHED: track 19.3 -> 21.8 mm
- net Net-(F1-Pad2): track 33.0 -> 31.9 mm

Commit message: chamfered the corners , so u kno its real
Other:
- outline, holes or cut-outs redrawn
Changed lines of the file:
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@@
     )
   )
-  (gr_rect (start 54.89899 41.694398) (end 104.675602 76.21101)
-    (stroke (width 0.1) (type default)) (fill none) (layer "Edge.Cuts"))
+  (gr_line (start 103.8 41.7) (end 103 41.7)
+    (stroke (width 0.1) (type default)) (layer "Edge.Cuts"))
+  (gr_line (start 103 41.7) (end 58.3 41.7)
+    (stroke (width 0.1) (type default)) (layer "Edge.Cuts"))
+  (gr_line (start 104.7 74.1) (end 104.7 43.4)
+    (stroke (width 0.1) (type default)) (layer "Edge.Cuts"))
+  (gr_line (start 104.3 41.7) (end 104.6 42)
+    (stroke (width 0.1) (type default)) (layer "Edge.Cuts"))
+  (gr_line (start 57.3 41.7) (end 55.2 43.8)
+    (stroke (width 0.1) (type default)) (layer "Edge.Cuts"))
+  (gr_line (start 103.8 41.7) (end 104.3 41.7)
+    (stroke (width 0.1) (type default)) (layer "Edge.Cuts"))
+  (gr_line (start 104.7 43.4) (end 104.7 42.6)
+    (stroke (width 0.1) (type default)) (layer "Edge.Cuts"))
+  (gr_line (start 54.9 44.1) (end 54.9 45.1)
+    (stroke (width 0.1) (type default)) (layer "Edge.Cuts"))
+  (gr_line (start 58 76.2) (end 102.6 76.2)
+    (stroke (width 0.1) (type default)) (layer "Edge.Cuts"))
+  (gr_line (start 104.6 42) (end 104.7 42.1)
+    (stroke (width 0.1) (type default)) (layer "Edge.Cuts"))
+  (gr_line (start 58.3 41.7) (end 57.3 41.7)
+    (stroke (width 0.1) (type default)) (layer "Edge.Cuts"))
+  (gr_line (start 102.6 76.2) (end 104.7 74.1)
+    (stroke (width 0.1) (type default)) (layer "Edge.Cuts"))
+  (gr_line (start 104.7 42.1) (end 104.7 42.6)
+    (stroke (width 0.1) (type default)) (layer "Edge.Cuts"))
+  (gr_line (start 54.9 45.1) (end 54.9 73.1)
+    (stroke (width 0.1) (type default)) (layer "Edge.Cuts"))
+  (gr_line (start 54.9 73.1) (end 58 76.2)
+    (stroke (width 0.1) (type default)) (layer "Edge.Cuts"))
+  (gr_line (start 55.2 43.8) (end 54.9 44.1)
+    (stroke (width 0.1) (type default)) (layer "Edge.Cuts"))
   (segment (start 102.81 42.17) (end 102.48 42.5) (width 0.508) (layer "F.Cu") (net 1))
   (segment (start 94.545 56.06) (end 98.2 56.06) (width 0.381) (layer "F.Cu") (net 1))
@@
   (via (at 103.515 47.65) (size 0.45) (drill 0.2) (layers "F.Cu" "B.Cu") (net 2))
   (via (at 88.53 49.755) (size 0.45) (drill 0.2) (layers "F.Cu" "B.Cu") (net 2))
-  (via (at 55.455 43.43) (size 0.45) (drill 0.2) (layers "F.Cu" "B.Cu") (net 2))
+  (via (at 57 42.9) (size 0.45) (drill 0.2) (layers "F.Cu" "B.Cu") (net 2))
   (via (at 100.525 51.69) (size 0.45) (drill 0.2) (layers "F.Cu" "B.Cu") (net 2))
   (via (at 103.35 52.755) (size 0.45) (drill 0.2) (layers "F.Cu" "B.Cu") (net 2))
@@
   (via (at 87.975884 50.203389) (size 0.45) (drill 0.2) (layers "F.Cu" "B.Cu") (net 2))
   (via (at 76.295 44.645) (size 0.45) (drill 0.2) (layers "F.Cu" "B.Cu") (net 2))
-  (via (at 55.8 42.59) (size 0.45) (drill 0.2) (layers "F.Cu" "B.Cu") (net 2))
+  (via (at 56.1 43.9) (size 0.45) (drill 0.2) (layers "F.Cu" "B.Cu") (net 2))
   (via (at 99.755 51.185) (size 0.45) (drill 0.2) (layers "F.Cu" "B.Cu") (net 2))
   (via (at 97.69 43.12) (size 0.45) (drill 0.2) (layers "F.Cu" "B.Cu") (net 2))
